File: IMU_Breakout_Board/IMU_Breakout_Board.kicad_pcb (KiCad board)
At the start: 2 copper layers, 27.9 x 18.7 mm, 6 parts, among them J1 Conn_01x06, U1 BMI270

Commit message: stretched top ground plane
Routing:
- net GND: vias 0 -> 2
Other:
- board size 27.9 x 18.7 mm -> 29 x 19.4 mm
Changed lines of the file:
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@@
   )
   (gr_rect (start 110.333078 80.264) (end 117.856 77.724) (layer "F.SilkS") (width 0.2) (fill none))
-  (gr_line (start 91.44 62.4205) (end 119.38 62.5475) (layer "Edge.Cuts") (width 0.1))
-  (gr_line (start 91.44 81.026) (end 91.44 62.4205) (layer "Edge.Cuts") (width 0.1))
-  (gr_line (start 119.38 81.153) (end 119.38 62.5475) (layer "Edge.Cuts") (width 0.1))
-  (gr_line (start 91.44 81.026) (end 119.38 81.153) (layer "Edge.Cuts") (width 0.1))
+  (gr_line (start 91.44 62.4205) (end 120.396 62.5475) (layer "Edge.Cuts") (width 0.1))
+  (gr_line (start 91.44 81.7245) (end 91.44 62.4205) (layer "Edge.Cuts") (width 0.1))
+  (gr_line (start 120.396 81.8515) (end 120.396 62.5475) (layer "Edge.Cuts") (width 0.1))
+  (gr_line (start 91.44 81.7245) (end 120.396 81.8515) (layer "Edge.Cuts") (width 0.1))
   (gr_text "GND" (at 97.568199 66.170193) (layer "F.SilkS")
     (effects (font (size 0.9 0.9) (thickness 0.1)))
@@
   (segment (start 94.776149 72.142543) (end 100.590543 72.142543) (width 0.25) (layer "F.Cu") (net 3))
   (segment (start 110.201555 65.278) (end 111.076079 66.152524) (width 0.25) (layer "F.Cu") (net 3))
+  (via (at 108.712 76.454) (size 0.8) (drill 0.4) (layers "F.Cu" "B.Cu") (free) (net 4))
+  (via (at 100.33 73.66) (size 0.8) (drill 0.4) (layers "F.Cu" "B.Cu") (free) (net 4))
   (segment (start 94.515606 79.502) (end 100.33 79.502) (width 0.25) (layer "F.Cu") (net 6))
   (segment (start 112.738579 67.315024) (end 113.532976 67.315024) (width 0.25) (layer "F.Cu") (net 6))
@@
     (polygon
       (pts
-        (xy 118.872 80.772)
-        (xy 91.948 80.772)
-        (xy 91.948 62.992)
-        (xy 118.872 62.992)
+        (xy 120.142 81.534)
+        (xy 91.694 81.534)
+        (xy 91.694 62.738)
+        (xy 120.142 62.738)
       )
     )

Commit message: final commit 3/16
Routing:
- net /IMU_A_INT1: track 39.1 -> 40.6 mm
- net /IMU_A_INT2: track 37.6 -> 38.8 mm
- net /IMU_A_SCL: track 68.6 -> 69.4 mm
Other:
- board text added: "IMU Breakout Board Rev 1.0 Space@VT Edited by: Kylie Angel"
- board text removed: "IMU Breakout Board Rev 1.0 Space@VT Edited by: Kylie A"
Changed lines of the file:
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@@
   )
   (setup
+    (stackup
+      (layer "F.SilkS" (type "Top Silk Screen"))
+      (layer "F.Paste" (type "Top Solder Paste"))
+      (layer "F.Mask" (type "Top Solder Mask") (thickness 0.01))
+      (layer "F.Cu" (type "copper") (thickness 0.035))
+      (layer "dielectric 1" (type "core") (thickness 1.51) (material "FR4") (epsilon_r 4.5) (loss_tangent 0.02))
+      (layer "B.Cu" (type "copper") (thickness 0.035))
+      (layer "B.Mask" (type "Bottom Solder Mask") (thickness 0.01))
+      (layer "B.Paste" (type "Bottom Solder Paste"))
+      (layer "B.SilkS" (type "Bottom Silk Screen"))
+      (copper_finish "None")
+      (dielectric_constraints no)
+    )
     (pad_to_mask_clearance 0)
     (pcbplotparams
@@
     )
   )
-  (gr_rect (start 110.333078 80.264) (end 117.856 77.724) (layer "F.SilkS") (width 0.2) (fill none))
+  (gr_rect (start 118.819289 80.329604) (end 117.041289 73.774143) (layer "F.SilkS") (width 0.2) (fill none))
   (gr_line (start 91.44 62.4205) (end 120.396 62.5475) (layer "Edge.Cuts") (width 0.1))
   (gr_line (start 91.44 81.7245) (end 91.44 62.4205) (layer "Edge.Cuts") (width 0.1))
@@
     (effects (font (size 0.9 0.9) (thickness 0.1)))
   )
-  (gr_text "IMU Breakout Board Rev 1.0\nSpace@VT\nEdited by: Kylie A" (at 114.135874 79.046711) (layer "F.SilkS")
-    (effects (font (size 0.3 0.3) (thickness 0.075)))
+  (gr_text "IMU Breakout Board Rev 1.0\nSpace@VT\nEdited by: Kylie Angel" (at 117.856 76.962 90) (layer "F.SilkS")
+    (effects (font (size 0.2 0.2) (thickness 0.05)))
   )
   (gr_text "+3.3V" (at 97.570114 68.758649) (layer "F.SilkS")
@@
   (via (at 100.33 76.708) (size 0.8) (drill 0.4) (layers "F.Cu" "B.Cu") (net 1))
   (via (at 116.332 63.754) (size 0.8) (drill 0.4) (layers "F.Cu" "B.Cu") (net 1))
-  (segment (start 118.11 65.532) (end 116.332 63.754) (width 0.25) (layer "B.Cu") (net 1))
+  (segment (start 99.06 77.978) (end 99.06 79.756) (width 0.25) (layer "B.Cu") (net 1))
   (segment (start 100.33 76.708) (end 99.06 77.978) (width 0.25) (layer "B.Cu") (net 1))
-  (segment (start 99.06 77.978) (end 99.06 79.756) (width 0.25) (layer "B.Cu") (net 1))
-  (segment (start 118.11 79.756) (end 118.11 65.532) (width 0.25) (layer "B.Cu") (net 1))
+  (segment (start 119.126 66.548) (end 116.332 63.754) (width 0.25) (layer "B.Cu") (net 1))
+  (segment (start 119.126 78.74) (end 119.126 66.548) (width 0.25) (layer "B.Cu") (net 1))
+  (segment (start 117.639489 80.226511) (end 119.126 78.74) (width 0.25) (layer "B.Cu") (net 1))
   (segment (start 99.06 79.756) (end 99.530511 80.226511) (width 0.25) (layer "B.Cu") (net 1))
-  (segment (start 117.639489 80.226511) (end 118.11 79.756) (width 0.25) (layer "B.Cu") (net 1))
   (segment (start 99.530511 80.226511) (end 117.639489 80.226511) (width 0.25) (layer "B.Cu") (net 1))
   (segment (start 115.567024 67.815024) (end 115.57 67.818) (width 0.25) (layer "F.Cu") (net 2))
   (segment (start 114.343812 73.92659) (end 112.324402 75.946) (width 0.25) (layer "F.Cu") (net 2))
   (segment (start 100.482341 69.540311) (end 94.713917 69.540311) (width 0.25) (layer "F.Cu") (net 2))
-  (segment (start 92.202 80.01) (end 92.62652 80.43452) (width 0.25) (layer "F.Cu") (net 2))
+  (segment (start 92.456 70.104) (end 92.202 70.358) (width 0.25) (layer "F.Cu") (net 2))
+  (segment (start 92.202 70.358) (end 92.202 80.01) (width 0.25) (layer "F.Cu") (net 2))
+  (segment (start 92.574692 70.104) (end 92.456 70.104) (width 0.25) (layer "F.Cu") (net 2))
   (segment (start 101.854 68.168652) (end 101.854 69.342) (width 0.25) (layer "F.Cu") (net 2))
+  (segment (start 92.202 80.01) (end 92.964 80.772) (width 0.25) (layer "F.Cu") (net 2))
   (segment (start 115.824 74.676) (end 115.824 71.12) (width 0.25) (layer "F.Cu") (net 2))
   (segment (start 112.738579 67.815024) (end 113.789024 67.815024) (width 0.25) (layer "F.Cu") (net 2))
   (segment (start 110.998 68.567125) (end 110.998 70.104) (width 0.25) (layer "F.Cu") (net 2))
-  (segment (start 92.62652 80.43452) (end 113.11348 80.43452) (width 0.25) (layer "F.Cu") (net 2))
+  (segment (start 115.824 77.724) (end 115.824 74.676) (width 0.25) (layer "F.Cu") (net 2))
   (segment (start 112.324402 75.946) (end 112.014 75.946) (width 0.25) (layer "F.Cu") (net 2))
-  (segment (start 92.574692 70.104) (end 92.456 70.104) (width 0.25) (layer "F.Cu") (net 2))
+  (segment (start 112.776 80.772) (end 115.824 77.724) (width 0.25) (layer "F.Cu") (net 2))
   (segment (start 104.14 65.882652) (end 101.854 68.168652) (width 0.25) (layer "F.Cu") (net 2))
   (segment (start 115.57 67.818) (end 115.57 65.532) (width 0.25) (layer "F.Cu") (net 2))
@@
   (segment (start 115.57 70.866) (end 111.76 70.866) (width 0.25) (layer "F.Cu") (net 2))
   (segment (start 111.076079 68.489046) (end 110.998 68.567125) (width 0.25) (layer "F.Cu") (net 2))
-  (segment (start 92.202 70.358) (end 92.202 80.01) (width 0.25) (layer "F.Cu") (net 2))
   (segment (start 115.824 71.12) (end 115.57 70.866) (width 0.25) (layer "F.Cu") (net 2))
   (segment (start 100.482341 69.540311) (end 102.496856 69.540311) (width 0.25) (layer "F.Cu") (net 2))
   (segment (start 102.496856 69.540311) (end 104.181335 71.22479) (width 0.25) (layer "F.Cu") (net 2))
-  (segment (start 113.11348 80.43452) (end 115.824 77.724) (width 0.25) (layer "F.Cu") (net 2))
   (segment (start 113.789024 67.815024) (end 115.567024 67.815024) (width 0.25) (layer "F.Cu") (net 2))
   (segment (start 94.713917 69.540311) (end 93.926149 68.752543) (width 0.25) (layer "F.Cu") (net 2))
-  (segment (start 92.456 70.104) (end 92.202 70.358) (width 0.25) (layer "F.Cu") (net 2))
   (segment (start 113.789024 68.836976) (end 111.76 70.866) (width 0.25) (layer "F.Cu") (net 2))
   (segment (start 110.538414 75.946) (end 108.601673 74.009259) (width 0.25) (layer "F.Cu") (net 2))
@@
   (segment (start 112.014 75.946) (end 114.554 75.946) (width 0.25) (layer "F.Cu") (net 2))
   (segment (start 93.926149 68.752543) (end 92.574692 70.104) (width 0.25) (layer "F.Cu") (net 2))
+  (segment (start 92.964 80.772) (end 112.776 80.772) (width 0.25) (layer "F.Cu") (net 2))
   (segment (start 111.076079 67.977524) (end 111.076079 68.489046) (width 0.25) (layer "F.Cu") (net 2))
-  (segment (start 115.824 77.724) (end 115.824 74.676) (width 0.25) (layer "F.Cu") (net 2))
   (segment (start 115.57 65.532) (end 115.062 65.024) (width 0.25) (layer "F.Cu") (net 2))
   (segment (start 110.998 70.104) (end 111.76 70.866) (width 0.25) (layer "F.Cu") (net 2))
@@
   (via (at 100.33 79.502) (size 0.8) (drill 0.4) (layers "F.Cu" "B.Cu") (net 6))
   (segment (start 100.33 79.502) (end 114.3 79.502) (width 0.25) (layer "B.Cu") (net 6))
-  (segment (start 116.84 69.088) (end 114.3 66.548) (width 0.25) (layer "B.Cu") (net 6))
-  (segment (start 114.3 79.502) (end 116.84 76.962) (width 0.25) (layer "B.Cu") (net 6))
-  (segment (start 116.84 76.962) (end 116.84 69.088) (width 0.25) (layer "B.Cu") (net 6))
+  (segment (start 114.3 79.502) (end 118.364 75.438) (width 0.25) (layer "B.Cu") (net 6))
+  (segment (start 118.364 70.612) (end 114.3 66.548) (width 0.25) (layer "B.Cu") (net 6))
+  (segment (start 118.364 75.438) (end 118.364 70.612) (width 0.25) (layer "B.Cu") (net 6))
   (segment (start 95.531606 77.978) (end 102.108 77.978) (width 0.25) (layer "F.Cu") (net 8))
   (segment (start 108.966 68.834) (end 109.728 69.596) (width 0.25) (layer "F.Cu") (net 8))
@@
   (via (at 109.728 69.596) (size 0.8) (drill 0.4) (layers "F.Cu" "B.Cu") (net 8))
   (via (at 102.108 77.978) (size 0.8) (drill 0.4) (layers "F.Cu" "B.Cu") (net 8))
+  (segment (start 117.602 72.136) (end 115.062 69.596) (width 0.25) (layer "B.Cu") (net 8))
+  (segment (start 115.062 69.596) (end 109.728 69.596) (width 0.25) (layer "B.Cu") (net 8))
   (segment (start 102.108 77.978) (end 114.3 77.978) (width 0.25) (layer "B.Cu") (net 8))
-  (segment (start 114.3 77.978) (end 115.824 76.454) (width 0.25) (layer "B.Cu") (net 8))
-  (segment (start 115.062 69.596) (end 109.728 69.596) (width 0.25) (layer "B.Cu") (net 8))
-  (segment (start 115.824 76.454) (end 115.824 70.358) (width 0.25) (layer "B.Cu") (net 8))
-  (segment (start 115.824 70.358) (end 115.062 69.596) (width 0.25) (layer "B.Cu") (net 8))
+  (segment (start 114.3 77.978) (end 117.602 74.676) (width 0.25) (layer "B.Cu") (net 8))
+  (segment (start 117.602 74.676) (end 117.602 72.136) (width 0.25) (layer "B.Cu") (net 8))
   (zone (net 4) (net_name "GND") (layers F&B.Cu) (hatch edge 0.508)
     (connect_pads (clearance 0.508))
@@
     )
   )
+  (group "" (id 238ea273-ed9a-4612-bbdf-9ad56281636a)
+    (members
+      5bb1348c-4f39-433e-acfc-4dde6d92f141
+      cdb3bb6c-9069-46af-90e1-884abbe27eee
+    )
+  )
   (group "" (id 5e4bed7f-1f28-41f8-9892-1ddfc9fc9aeb)
     (members
@@
     )
   )
-  (group "" (id c17f9a6e-6669-4413-9c98-da8cfab7ee0c)
-    (members
-      5bb1348c-4f39-433e-acfc-4dde6d92f141
-      cdb3bb6c-9069-46af-90e1-884abbe27eee
-    )
-  )
