File: IMU_BB_Rev2/IMU_BB_Rev2.kicad_pcb (KiCad board)
At the start: 2 copper layers, 13 x 8 mm, 6 parts, among them J1 Conn_01x04, U1 BMI270

Commit message: 3/17
Parts:
- moved R1 2.20 mm to (71.8, 61.5)
- moved R2 1.22 mm to (70.2, 61.5)
- moved J1 0.07 mm to (79.1, 57.7)
Routing:
- net /IMU_A_SCL: track 0.00 -> 14.7 mm
- net /IMU_A_SDA: track 0.00 -> 11.4 mm
- added copper zone on In2.Cu, net +3V3
- added copper zone on B.Cu, net GND
- added copper zone on F.Cu, net GND
Other:
- copper layers 2 -> 4
Changed lines of the file:
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@@
 (kicad_pcb (version 20211014) (generator pcbnew)
   (general
-    (thickness 1.6)
+    (thickness 1.724)
   )
   (paper "A5")
   (layers
     (0 "F.Cu" signal)
+    (1 "In1.Cu" signal)
+    (2 "In2.Cu" signal)
     (31 "B.Cu" signal)
     (32 "B.Adhes" user "B.Adhesive")
@@
   )
   (setup
+    (stackup
+      (layer "F.SilkS" (type "Top Silk Screen"))
+      (layer "F.Paste" (type "Top Solder Paste"))
+      (layer "F.Mask" (type "Top Solder Mask") (thickness 0.01))
+      (layer "F.Cu" (type "copper") (thickness 0.035))
+      (layer "dielectric 1" (type "core") (thickness 0.2) (material "FR4") (epsilon_r 4.5) (loss_tangent 0.02))
+      (layer "In1.Cu" (type "copper") (thickness 0.017))
+      (layer "dielectric 2" (type "prepreg") (thickness 1.2) (material "FR4") (epsilon_r 4.5) (loss_tangent 0.02))
+      (layer "In2.Cu" (type "copper") (thickness 0.017))
+      (layer "dielectric 3" (type "core") (thickness 0.2) (material "FR4") (epsilon_r 4.5) (loss_tangent 0.02))
+      (layer "B.Cu" (type "copper") (thickness 0.035))
+      (layer "B.Mask" (type "Bottom Solder Mask") (thickness 0.01))
+      (layer "B.Paste" (type "Bottom Solder Paste"))
+      (layer "B.SilkS" (type "Bottom Silk Screen"))
+      (copper_finish "None")
+      (dielectric_constraints no)
+    )
     (pad_to_mask_clearance 0)
     (pcbplotparams
@@
   )
   (footprint "Resistor_SMD:R_0603_1608Metric" (layer "F.Cu")
-    (at 71.4 61.64 90)
+    (at 70.18 61.53 90)
     (descr "Resistor SMD 0603 (1608 Metric), square (rectangular) end terminal, IPC_7351 nominal, (Body size source: IPC-SM-782 page 72, https://www.pcb-3d.com/wordpress/wp-content/uploads/ipc-sm-782a_amendment_1_and_2.pdf), generated with kicad-footprint-generator")
     (tags "resistor")
@@
   )
   (footprint "Resistor_SMD:R_0603_1608Metric" (layer "F.Cu")
-    (at 69.58 61.68 90)
+    (at 71.77 61.49 90)
     (descr "Resistor SMD 0603 (1608 Metric), square (rectangular) end terminal, IPC_7351 nominal, (Body size source: IPC-SM-782 page 72, https://www.pcb-3d.com/wordpress/wp-content/uploads/ipc-sm-782a_amendment_1_and_2.pdf), generated with kicad-footprint-generator")
     (tags "resistor")
@@
   )
   (footprint "Connector_PinHeader_3.00mm:PinHeader_1x04_P3.00mm_Vertical" (layer "F.Cu")
-    (at 79.01 57.64 -90)
+    (at 79.06 57.69 -90)
     (descr "Through hole straight pin header, 1x04, 2.54mm pitch, single row")
     (tags "Through hole pin header THT 1x04 2.54mm single row")
@@
   (gr_line (start 68.011 63.92) (end 80.969 63.96) (layer "Edge.Cuts") (width 0.1))
   (gr_line (start 68.072 55.94) (end 81.03 55.98) (layer "Edge.Cuts") (width 0.1))
-  (gr_text "GND" (at 78.99 59.56) (layer "F.SilkS")
+  (gr_text "GND" (at 79.04 59.61) (layer "F.SilkS")
     (effects (font (size 0.5 0.5) (thickness 0.075)))
   )
-  (gr_text "SCL" (at 72.89 59.52) (layer "F.SilkS")
+  (gr_text "SCL" (at 72.94 59.57) (layer "F.SilkS")
     (effects (font (size 0.5 0.5) (thickness 0.075)))
   )
-  (gr_text "SDA" (at 69.78 59.5) (layer "F.SilkS")
+  (gr_text "SDA" (at 69.83 59.55) (layer "F.SilkS")
     (effects (font (size 0.5 0.5) (thickness 0.075)))
   )
-  (gr_text "+3.3V" (at 75.94 59.54) (layer "F.SilkS")
+  (gr_text "+3.3V" (at 75.99 59.59) (layer "F.SilkS")
     (effects (font (size 0.5 0.5) (thickness 0.075)))
   )
+  (segment (start 74.52 60.185978) (end 74.52 60.6975) (width 0.25) (layer "F.Cu") (net 1))
+  (segment (start 76.32 63.18) (end 76.63 62.87) (width 0.25) (layer "F.Cu") (net 1))
+  (segment (start 71.5 62.215) (end 71.515 62.215) (width 0.25) (layer "F.Cu") (net 1))
+  (segment (start 72.53 58.124) (end 72.964 57.69) (width 0.25) (layer "F.Cu") (net 1))
+  (segment (start 72.48 63.18) (end 76.32 63.18) (width 0.25) (layer "F.Cu") (net 1))
+  (segment (start 74.885978 59.611978) (end 74.885978 59.82) (width 0.25) (layer "F.Cu") (net 1))
+  (segment (start 76.14 59.82) (end 74.885978 59.82) (width 0.25) (layer "F.Cu") (net 1))
+  (segment (start 71.515 62.215) (end 72.48 63.18) (width 0.25) (layer "F.Cu") (net 1))
+  (segment (start 76.63 60.31) (end 76.14 59.82) (width 0.25) (layer "F.Cu") (net 1))
+  (segment (start 74.885978 59.82) (end 74.52 60.185978) (width 0.25) (layer "F.Cu") (net 1))
+  (segment (start 72.964 57.69) (end 74.885978 59.611978) (width 0.25) (layer "F.Cu") (net 1))
+  (segment (start 76.63 62.87) (end 76.63 60.31) (width 0.25) (layer "F.Cu") (net 1))
+  (segment (start 73.91 59.75) (end 69.97 59.75) (width 0.25) (layer "F.Cu") (net 3))
+  (segment (start 69.555 62.355) (end 69.38048 62.18048) (width 0.25) (layer "F.Cu") (net 3))
+  (segment (start 69.38048 62.18048) (end 69.38048 59.11952) (width 0.25) (layer "F.Cu") (net 3))
+  (segment (start 69.38048 59.11952) (end 69.38048 58.22552) (width 0.25) (layer "F.Cu") (net 3))
+  (segment (start 74.02 60.6975) (end 74.02 59.86) (width 0.25) (layer "F.Cu") (net 3))
+  (segment (start 69.38048 59.16048) (end 69.38048 59.11952) (width 0.25) (layer "F.Cu") (net 3))
+  (segment (start 74.02 59.86) (end 73.91 59.75) (width 0.25) (layer "F.Cu") (net 3))
+  (segment (start 69.97 59.75) (end 69.38048 59.16048) (width 0.25) (layer "F.Cu") (net 3))
+  (segment (start 70.18 62.355) (end 69.555 62.355) (width 0.25) (layer "F.Cu") (net 3))
+  (segment (start 69.38048 58.22552) (end 69.916 57.69) (width 0.25) (layer "F.Cu") (net 3))
+  (zone (net 4) (net_name "GND") (layers F&B.Cu) (hatch edge 0.508)
+    (connect_pads (clearance 0.508))
+    (min_thickness 0.254) (filled_areas_thickness no)
+    (fill yes (thermal_gap 0.508) (thermal_bridge_width 0.508))
+    (polygon
+      (pts
+        (xy 80.85 56.12)
+        (xy 80.85 63.76)
+        (xy 68.2 63.76)
+        (xy 68.23 56.09)
+      )
+    )
+  )
+  (zone (net 2) (net_name "+3V3") (layer "In2.Cu") (hatch edge 0.508)
+    (connect_pads (clearance 0.508))
+    (min_thickness 0.254) (filled_areas_thickness no)
+    (fill yes (thermal_gap 0.508) (thermal_bridge_width 0.508))
+    (polygon
+      (pts
+        (xy 80.85 56.12)
+        (xy 80.75 63.72)
+        (xy 68.2 63.62)
+        (xy 68.23 56.09)
+      )
+    )
+  )
   (group "" (id e8ae8aa2-6c83-4751-87be-af18c04f637b)

Commit message: 3/18 Needs checking
Routing:
- added copper zone on In1.Cu, net GND
- removed copper zone on B.Cu, net GND
- removed copper zone on F.Cu, net GND
Other:
- board text added: "IMU Breakout Board Rev 2.0 Edited by Kylie Angel"
Changed lines of the file:
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@@
 (kicad_pcb (version 20211014) (generator pcbnew)
   (general
-    (thickness 1.724)
+    (thickness 1.76)
   )
   (paper "A5")
@@
       (layer "F.Cu" (type "copper") (thickness 0.035))
       (layer "dielectric 1" (type "core") (thickness 0.2) (material "FR4") (epsilon_r 4.5) (loss_tangent 0.02))
-      (layer "In1.Cu" (type "copper") (thickness 0.017))
+      (layer "In1.Cu" (type "copper") (thickness 0.035))
       (layer "dielectric 2" (type "prepreg") (thickness 1.2) (material "FR4") (epsilon_r 4.5) (loss_tangent 0.02))
-      (layer "In2.Cu" (type "copper") (thickness 0.017))
+      (layer "In2.Cu" (type "copper") (thickness 0.035))
       (layer "dielectric 3" (type "core") (thickness 0.2) (material "FR4") (epsilon_r 4.5) (loss_tangent 0.02))
       (layer "B.Cu" (type "copper") (thickness 0.035))
@@
   (gr_line (start 68.011 63.92) (end 80.969 63.96) (layer "Edge.Cuts") (width 0.1))
   (gr_line (start 68.072 55.94) (end 81.03 55.98) (layer "Edge.Cuts") (width 0.1))
+  (gr_text "IMU Breakout Board Rev 2.0\nEdited by Kylie Angel" (at 68.79 62.35 90) (layer "F.SilkS")
+    (effects (font (size 0.1 0.1) (thickness 0.025)))
+  )
   (gr_text "GND" (at 79.04 59.61) (layer "F.SilkS")
     (effects (font (size 0.5 0.5) (thickness 0.075)))
@@
   (segment (start 70.18 62.355) (end 69.555 62.355) (width 0.25) (layer "F.Cu") (net 3))
   (segment (start 69.38048 58.22552) (end 69.916 57.69) (width 0.25) (layer "F.Cu") (net 3))
-  (zone (net 4) (net_name "GND") (layers F&B.Cu) (hatch edge 0.508)
+  (zone (net 4) (net_name "GND") (layer "In1.Cu") (hatch edge 0.508)
     (connect_pads (clearance 0.508))
     (min_thickness 0.254) (filled_areas_thickness no)

Commit message: 3/19
Parts:
- moved C1 0.21 mm to (79.5, 61.6)
- moved J1 0.11 mm to (79.0, 57.6)
Routing:
- net GND: track 0.00 -> 11.8 mm, vias 0 -> 2
- net +3V3: track 0.00 -> 11.3 mm, vias 0 -> 3
- net /IMU_A_SCL: track 14.7 -> 12.1 mm, vias 0 -> 2

Commit message: final commit
Routing:
- net /IMU_A_SCL: track 12.1 -> 11.5 mm
Other:
- outline, holes or cut-outs redrawn
Changed lines of the file:
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@@
       (layerselection 0x00010fc_ffffffff)
       (disableapertmacros false)
-      (usegerberextensions false)
+      (usegerberextensions true)
       (usegerberattributes true)
       (usegerberadvancedattributes true)
@@
       (plotinvisibletext false)
       (sketchpadsonfab false)
-      (subtractmaskfromsilk false)
+      (subtractmaskfromsilk true)
       (outputformat 1)
       (mirror false)
-      (drillshape 1)
+      (drillshape 0)
       (scaleselection 1)
-      (outputdirectory "")
+      (outputdirectory "Gerbers_Drill_files/")
     )
   )
@@
       (net 3 "/IMU_A_SDA") (pinfunction "SDX") (pintype "bidirectional"))
   )
-  (gr_line (start 81.03 56.02) (end 80.99 63.96) (layer "Edge.Cuts") (width 0.1))
-  (gr_line (start 68.03 55.94) (end 67.99 63.88) (layer "Edge.Cuts") (width 0.1))
-  (gr_line (start 68.011 63.92) (end 80.969 63.96) (layer "Edge.Cuts") (width 0.1))
-  (gr_line (start 68.072 55.94) (end 81.03 55.98) (layer "Edge.Cuts") (width 0.1))
+  (gr_line (start 81 55.96) (end 80.99 63.94) (layer "Edge.Cuts") (width 0.1))
+  (gr_line (start 68.02 55.95) (end 67.98 63.93) (layer "Edge.Cuts") (width 0.1))
+  (gr_line (start 67.98 63.93) (end 80.99 63.94) (layer "Edge.Cuts") (width 0.1))
+  (gr_line (start 68.02 55.95) (end 81 55.96) (layer "Edge.Cuts") (width 0.1))
   (gr_text "IMU Breakout Board Rev 2.0\nEdited by Kylie Angel" (at 68.45 62.31 90) (layer "F.SilkS")
     (effects (font (size 0.1 0.1) (thickness 0.025)))
@@
   (segment (start 74.585106 59.629859) (end 74.585106 59.311106) (width 0.2) (layer "F.Cu") (net 1))
   (segment (start 74.585106 59.629859) (end 74.585106 60.632394) (width 0.2) (layer "F.Cu") (net 1))
-  (segment (start 72.53 58.124) (end 72.964 57.69) (width 0.25) (layer "F.Cu") (net 1))
+  (segment (start 71.77 62.315) (end 71.77 62.47) (width 0.2) (layer "F.Cu") (net 1))
   (segment (start 74.585106 60.632394) (end 74.52 60.6975) (width 0.2) (layer "F.Cu") (net 1))
-  (segment (start 71.77 62.315) (end 71.77 62.47) (width 0.2) (layer "F.Cu") (net 1))
   (segment (start 74.585106 59.311106) (end 72.964 57.69) (width 0.2) (layer "F.Cu") (net 1))
   (segment (start 71.77 62.47) (end 70.96 63.28) (width 0.2) (layer "F.Cu") (net 1))
   (via (at 70.96 63.28) (size 0.6) (drill 0.3) (layers "F.Cu" "B.Cu") (net 1))
   (via (at 74.585106 59.629859) (size 0.6) (drill 0.3) (layers "F.Cu" "B.Cu") (net 1))
-  (segment (start 71.409511 62.830489) (end 73.619511 62.830489) (width 0.2) (layer "In1.Cu") (net 1))
-  (segment (start 73.619511 62.830489) (end 74.585106 61.864894) (width 0.2) (layer "In1.Cu") (net 1))
-  (segment (start 70.96 63.28) (end 71.409511 62.830489) (width 0.2) (layer "In1.Cu") (net 1))
-  (segment (start 74.585106 61.864894) (end 74.585106 59.629859) (width 0.2) (layer "In1.Cu") (net 1))
+  (segment (start 73.264096 63.18) (end 71.06 63.18) (width 0.2) (layer "In1.Cu") (net 1))
+  (segment (start 71.06 63.18) (end 70.96 63.28) (width 0.2) (layer "In1.Cu") (net 1))
+  (segment (start 73.264096 63.18) (end 74.585106 61.85899) (width 0.2) (layer "In1.Cu") (net 1))
+  (segment (start 74.585106 61.85899) (end 74.585106 59.629859) (width 0.2) (layer "In1.Cu") (net 1))
   (segment (start 70.96 63.28) (end 71 63.24) (width 0.2) (layer "B.Cu") (net 1))
   (segment (start 71.77 60.42) (end 71.77 60.665) (width 0.2) (layer "F.Cu") (net 2))
@@
   (segment (start 77.51 62.455) (end 77.51 63.19) (width 0.2) (layer "F.Cu") (net 4))
   (segment (start 75.44952 63.28048) (end 77.41952 63.28048) (width 0.2) (layer "F.Cu") (net 4))
-  (segment (start 72.83 59.84) (end 72.83 59.71) (width 0.2) (layer "F.Cu") (net 4))
   (via (at 72.83 59.84) (size 0.6) (drill 0.3) (layers "F.Cu" "B.Cu") (net 4))
   (via (at 76.5 63.26) (size 0.6) (drill 0.3) (layers "F.Cu" "B.Cu") (net 4))
